Commit message: added pointcloud-to-ocgrid package and set up

File: platypus_gazebo/urdf/platypus.xacro (robot description, xacro)
@@ -243,5 +243,5 @@
     <parent link="board"/>
     <child link="lidar_base" />
-    <origin xyz="0.2 0 0" rpy="0 0 0"/>
+    <origin xyz="0.15 0 0" rpy="0 0 0"/>
   </joint>
   <link name="lidar_base">
